File: card.sch (KiCad schematic (older format))
At the start: 7 parts, among them CON1 USB-MINI-B, IC1 ATTINY44-S, P1 CONN_3X2

Commit message: working attiny26 rev sent to oshpark
Parts:
- removed IC1: ATTINY44-S, SO14, symbol ATTINY44-S
- added IC1: ATTINY26-S, Housings_SOIC:SOIC-20_7.5x12.8mm_Pitch1.27mm, symbol ATTINY26-S
- added R2: 4.7k, Resistors_SMD:R_0603_HandSoldering, symbol R-RESCUE-card
- C1: footprint ~ -> Capacitors_SMD:C_0603_HandSoldering; symbol C -> C-RESCUE-card
- CON1: footprint (none) -> card:15542661MicroUSBB
- D1: footprint ~ -> card:SMini4-F3-B
- P1: footprint (none) -> Pin_Headers:Pin_Header_Straight_2x03
- R1: footprint ~ -> Resistors_SMD:R_0603_HandSoldering; symbol R -> R-RESCUE-card
- RP1: footprint ~ -> card:MNR12
Connections:
- net labels added: A, B, Down, Left, Right, Select, Start, Up
- wire segments 56 -> 49
Other:
- moved on the sheet: C1, CON1, D1, R1, RP1
